File: electronics/pico-joystick.kicad_pcb (KiCad board)
At the start: 2 copper layers, 50 x 70 mm, 14 parts, among them J1 Gameport socket, J3 Serial, J4 Debug, U1 Raspberry Pi Pico

Commit message: Corrected PCB design
Parts:
- moved U1 55.2 mm to (141.8, 60.8), turned to 0 degrees
- moved J2 44.4 mm to (134.7, 100.5), turned to 90 degrees
- moved C1 36.0 mm to (168.1, 73.7)
- moved R1 36.0 mm to (168.1, 90.2)
- moved R4 36.0 mm to (168.1, 106.7)
- moved C2 35.4 mm to (172.6, 73.7)
- moved R2 35.4 mm to (172.6, 90.2)
- moved R3 35.4 mm to (172.6, 106.7)
- moved J3 35.2 mm to (135.2, 85.2), turned to 180 degrees
- renumbered J4 to J2, R3 to R1, R4 to R2, R1 to R3, R2 to R4
Connections:
- J1 pad 0: (no net) -> GND
- U1 pad 13: unconnected-(U1-GND-Pad13) -> GND
- U1 pad 18: unconnected-(U1-GND-Pad18) -> GND
- U1 pad 23: unconnected-(U1-GND-Pad23) -> GND
- U1 pad 28: unconnected-(U1-GND-Pad28) -> GND
- U1 pad 3: unconnected-(U1-GND-Pad3) -> GND
- U1 pad 33: unconnected-(U1-GND-Pad33) -> GND
- U1 pad 8: unconnected-(U1-GND-Pad8) -> GND
Routing:
- net Net-(J2-Pin_4): track 39.1 -> 115.7 mm, vias 1 -> 3
- net Net-(J1-Pad7): track 35.3 -> 84.4 mm, vias 2 -> 0
- net Net-(U1-GP17): track 14.8 -> 41.7 mm, vias 0 -> 1
- net +3V3: track 26.9 -> 52.5 mm, vias 0 -> 3
- net Net-(U1-GP16): track 19.7 -> 41.3 mm
- net Net-(U1-GP27): track 42.4 -> 62.3 mm, vias 1 -> 2
- net Net-(J2-Pin_3): track 30.3 -> 48.2 mm
- net Net-(J1-Pad2): track 48.1 -> 34.8 mm, vias 0 -> 1
- net Net-(U1-GP26): track 46.0 -> 58.1 mm, vias 0 -> 2
- net Net-(J2-Pin_2): track 26.7 -> 35.0 mm, vias 0 -> 2
- net Net-(J2-Pin_1): track 23.2 -> 27.7 mm
- net Net-(J3-Pin_4): track 15.2 -> 18.9 mm
- net Net-(J3-Pin_5): track 15.1 -> 18.6 mm
Other:
- board text added: "Pico Joystick v1.1"
- board text removed: "Pico Joystick v1.0"
